File: PCB/V1.1/BottleBuddy-V1.1.sch (EAGLE design)
At the start: 55 parts, among them Q1 MOSFET-PCHANNEL, Q2 MOSFET-PCHANNEL, Q3 200mA/50V, U1 74AHC1G125, U2 MAX1704X, U3 MMA8452Q, U4 BME280, U5 MCKPT-G1210-3916

Commit message: Modified V1.1 to use plug-in modules for Accelerometer and BME280 to make life easier.
Removed one LED.

Changed keep awake, moved DB18B20 so it can be close to the load cell and possibly fixed as it's by the fixed part.
Parts:
- removed C3, C5: 0.1uF, SparkFun-Capacitors:CAP0805
- removed C4: 4.7uF, SparkFun-Capacitors:CAP0805
- removed D3: RED, SparkFun-LED:LED1206
- removed Q2: MOSFET-PCHANNEL, SparkFun-DiscreteSemi:MOSFET-PCHANNEL
- removed R11: DNP, SparkFun-Resistors:RESISTOR1206
- removed R16: 10k, SparkFun-Resistors:RESISTOR1206
- removed R17: 100k, SparkFun-Resistors:RESISTOR1206
- removed R6: 1k5, SparkFun-Resistors:RESISTOR1206
- removed R8: 100r, SparkFun-Resistors:RESISTOR1206
- removed U3: MMA8452Q, SparkFun-Sensors:MMA8452Q
- removed U4: BME280, SparkFun-Sensors:BME280
- added 3V3_LOWER_TP, GND24, GND_LOWER_TP: TPTP20R, testpad:TPTP20R
- added BME280: (no value), SparkFun-Connectors:M06SILK_FEMALE_PTH
- added JP1: (no value), SparkFun-Connectors:M03PTH
- added LOGO1: OSHW-LOGOL, SparkFun-Aesthetics:OSHW-LOGOL
- added MMA8452Q: (no value), SparkFun-Connectors:M08SILK_FEMALE_PTH
- added R18: 10k, SparkFun-Resistors:RESISTOR1206
- added R19: 2k2, SparkFun-Resistors:RESISTOR1206
- added R21: DNP, SparkFun-Resistors:RESISTOR1206
- added RSTPDN: NFC IRQ, testpad:TPTP20R
- added SJ1: (no value), jumper:SJ
- R1, R9: value 100r -> 100R
- R10: value 10k -> 1k
- R12: value 10k -> 1M
- R2, R5: value (none) -> 30k
Connections:
- removed net INT2: U$1G$1.RX, U3.INT2
- removed net N$13: D3.A, R6.2
- removed net N$8: R6.1, U$1G$1.A4
- removed net NFC_POWER: Q2.G, R11.2, R16.1, R8.2
- new net N$20: MMA8452Q.6, R21.2
- new net RSTPDN: R19.2, RSTPDN.TP, U$1G$1.D4
- net 3.3V: now also 3V3_LOWER_TP.TP, BME280.2, BME280.6, JP5.2, MMA8452Q.2, R18.1, R21.1, SJ1.2; no longer C4.1, C5.1, Q2.S, R16.2, U3.SA0, U3.VDD, U3.VDDIO, U4.!CS, U4.VDD, U4.VDDIO
- net BUZZER: now also U$1G$1.A4; no longer U$1G$1.TX
- net GND: now also BME280.1, BME280.5, GND24.TP, GND_LOWER_TP.TP, JP1.1, MMA8452Q.3, R19.1; no longer C3.2, C4.2, C5.2, D3.C, R11.1, R17.2, U3.GND@0, U3.GND@1, U3.GND@2, U4.GND, U4.SDO/ADR
- net INT1: now also MMA8452Q.8; no longer U3.INT1
- net N$12: no longer R17.1
- net N$18: now also MMA8452Q.1, SJ1.1; no longer C3.1, U3.BYP
- net N$4: now also JP1.3, U$1G$1.RX; no longer JP5.2, Q2.D
- net N$7: now also JP1.2, U$1G$1.TX; no longer R8.1, U$1G$1.D4
- net SCALE_CLOCK: now also R18.2
- net SCL: now also BME280.4, MMA8452Q.4; no longer U3.SCL, U4.SCK/SCL
- net SDA: now also BME280.3, MMA8452Q.5; no longer U3.SDA, U4.SDI/SDA
Other:
- note added: "Addr: Fit R21 (0R): 0x1D DNP R21: 0x1C (SA low) NB: Board has 1k pulldown so with R21 fitted consumes 3mA."
- note added: "BME280"
- note added: "R18 - keep the scale in low power mode when CPU shutdown"
- note added: "Stephen Harrison"
- note added: "TODO: R19 - Can this be higher than 1k5 (10k too high) NFC reader has 10k pull-up. Perhaps remove that?"
- note added: "V1.1"
- note added: "http://www.ebay.co.uk/itm/MMA8452-Three-Axis-Accelerator-Module-PIC-ARM-Pi-Arduino-New-UK-Stock-UK-Seller-/201495494714?var=&hash=item2eea11403a:m:miFNPKejG0VKZeNKhIcq8lA"
- note removed: "Addr: 0x1C"
- moved on the sheet: 3V3, D1, KEEP_AWAKE, R13, R9
